File: auto_probe_pcb_outputs/pinout_grouped - Copy_probe_pcb.kicad_pcb (KiCad board)
At the start: 2 copper layers, 8.2 x 5.2 mm, 0 parts

Commit message: kicad script done?
Other:
- board text added: "CHIP_ID<0>"
- board text added: "CHIP_ID<1>"
- board text added: "CHIP_ID<2>"
- board text added: "CLKEXTM<0>"
- board text added: "CLKEXTM<1>"
- board text added: "CLKEXTP<0>"
- board text added: "CLKEXTP<1>"
- board text added: "CLKOUTN_MUX"
- board text added: "CLKOUTP_MUX"
- board text added: "CSB"
- board text added: "DFT_SCAN_SDI<1>"
- board text added: "DFT_SCAN_SDI<2>"
- board text added: "DFT_SCN_SDO<1>"
- board text added: "DFT_SCN_SDO<2>"
- board text added: "F"
- board text added: "LB_PCLK"
- board text added: "LED_I0_CURRENT"
- board text added: "LED_I0_SNS"
- board text added: "LED_I1_SNS"
- board text added: "RESET_N"
- board text added: "REXT1"
- board text added: "REXT2"
- board text added: "RSSI_L"
- board text added: "RSSI_R"
- board text added: "SCAN_CLK"
- board text added: "SCAN_EN"
- board text added: "SCAN_MODE"
- board text added: "SCAN_SAFE_MODE"
- board text added: "SCK"
- board text added: "SCL"
- board text added: "SDA"
- board text added: "SDI"
- board text added: "SEL_APB_SPI_N"
- board text added: "TEST_DLL_DESKEW_CKOUT"
- board text added: "TEST_LED_STRB0_CKOUT"
- board text added: "TEST_PLL4_CKOUT"
- board text added: "TEST_TX_CKOUT"
- board text added: "V3_CHIP ID<0>"
- board text added: "V3_CHIP ID<1>"
- board text added: "VATB_DLL"
- board text added: "VATB_LED0"
- board text added: "VATB_LED1"
- board text added: "VATB_RSSI0"
- board text added: "VATB_RSSI1"
- board text added: "VATB_TIA"
- board text added: "VDD08"
- board text added: "VDD08BIAS<0>"
- board text added: "VDD08D"
- board text added: "VDD08DLL<0>"
- board text added: "VDD08DLL<1>"
- board text added: "VDD08DLL<2>"
- board text added: "VDD08DLL<3>"
- board text added: "VDD08DLL<6>"
- board text added: "VDD08DLL<7>"
- board text added: "VDD08D_SNS"
- board text added: "VDD08LED"
- board text added: "VDD08PA"
- board text added: "VDD08PA_SNS"
- board text added: "VDD08TIA"
- board text added: "VDD08TIA_SNS"
- board text added: "VDD12LED"
- board text added: "VDD18A"
- board text added: "VDD18B"
- board text added: "VDD18C"
- board text added: "VDD18D"
- board text added: "VDD18E"
- board text added: "VDD18LED"
- board text added: "VDD18PLL<0>"
- board text added: "VDD18PLL<1>"
- board text added: "VDD18PLL<2>"
- board text added: "VDD18PLL<3>"
- board text added: "VDD18PLL<6>"
- board text added: "VDD18PLL<7>"
- board text added: "VDD18_BG<0>"
- board text added: "VDD50LED"
- board text added: "VDD50LED_SNS"
- board text added: "VDD50PD"
- board text added: "VDDDRVLED_SNS"
- board text added: "VDDLED_SNS"
- board text added: "VDDPST"
- board text added: "VSS"
- board text added: "VSSLED"
- board text added: "VSSPST"
- board text added: "VSSTIA"

Commit message: altium script
Other:
- board text removed: "CHIP_ID<0>"
- board text removed: "CHIP_ID<1>"
- board text removed: "CHIP_ID<2>"
- board text removed: "CLKEXTM<0>"
- board text removed: "CLKEXTM<1>"
- board text removed: "CLKEXTP<0>"
- board text removed: "CLKEXTP<1>"
- board text removed: "CLKOUTN_MUX"
- board text removed: "CLKOUTP_MUX"
- board text removed: "CSB"
- board text removed: "DFT_SCAN_SDI<1>"
- board text removed: "DFT_SCAN_SDI<2>"
- board text removed: "DFT_SCN_SDO<1>"
- board text removed: "DFT_SCN_SDO<2>"
- board text removed: "F"
- board text removed: "LB_PCLK"
- board text removed: "LED_I0_CURRENT"
- board text removed: "LED_I0_SNS"
- board text removed: "LED_I1_SNS"
- board text removed: "RESET_N"
- board text removed: "REXT1"
- board text removed: "REXT2"
- board text removed: "RSSI_L"
- board text removed: "RSSI_R"
- board text removed: "SCAN_CLK"
- board text removed: "SCAN_EN"
- board text removed: "SCAN_MODE"
- board text removed: "SCAN_SAFE_MODE"
- board text removed: "SCK"
- board text removed: "SCL"
- board text removed: "SDA"
- board text removed: "SDI"
- board text removed: "SEL_APB_SPI_N"
- board text removed: "TEST_DLL_DESKEW_CKOUT"
- board text removed: "TEST_LED_STRB0_CKOUT"
- board text removed: "TEST_PLL4_CKOUT"
- board text removed: "TEST_TX_CKOUT"
- board text removed: "V3_CHIP ID<0>"
- board text removed: "V3_CHIP ID<1>"
- board text removed: "VATB_DLL"
- board text removed: "VATB_LED0"
- board text removed: "VATB_LED1"
- board text removed: "VATB_RSSI0"
- board text removed: "VATB_RSSI1"
- board text removed: "VATB_TIA"
- board text removed: "VDD08"
- board text removed: "VDD08BIAS<0>"
- board text removed: "VDD08D"
- board text removed: "VDD08DLL<0>"
- board text removed: "VDD08DLL<1>"
- board text removed: "VDD08DLL<2>"
- board text removed: "VDD08DLL<3>"
- board text removed: "VDD08DLL<6>"
- board text removed: "VDD08DLL<7>"
- board text removed: "VDD08D_SNS"
- board text removed: "VDD08LED"
- board text removed: "VDD08PA"
- board text removed: "VDD08PA_SNS"
- board text removed: "VDD08TIA"
- board text removed: "VDD08TIA_SNS"
- board text removed: "VDD12LED"
- board text removed: "VDD18A"
- board text removed: "VDD18B"
- board text removed: "VDD18C"
- board text removed: "VDD18D"
- board text removed: "VDD18E"
- board text removed: "VDD18LED"
- board text removed: "VDD18PLL<0>"
- board text removed: "VDD18PLL<1>"
- board text removed: "VDD18PLL<2>"
- board text removed: "VDD18PLL<3>"
- board text removed: "VDD18PLL<6>"
- board text removed: "VDD18PLL<7>"
- board text removed: "VDD18_BG<0>"
- board text removed: "VDD50LED"
- board text removed: "VDD50LED_SNS"
- board text removed: "VDD50PD"
- board text removed: "VDDDRVLED_SNS"
- board text removed: "VDDLED_SNS"
- board text removed: "VDDPST"
- board text removed: "VSS"
- board text removed: "VSSLED"
- board text removed: "VSSPST"
- board text removed: "VSSTIA"
